File: pcb/keyboard-x2-lumberjack-arm-fancy.kicad_sch (KiCad schematic)
At the start: 13 parts, among them J1 16-pin USB-C Connector SMD, U1 STM32F103 Bluepill, or MiniF4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, U2 SN74LVC1T45DBV

Commit message: kicad: fix mounting hole
Parts:
- H5: footprint ProjectLocal:H_M2_Spacer_Hole -> ProjectLocal:H_M2_GH60_MountingHole
Changed lines of the file:
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@@
       (effects (font (size 1.27 1.27)) (justify left))
     )
-    (property "Footprint" "ProjectLocal:H_M2_Spacer_Hole" (id 2) (at 48.26 179.07 0)
+    (property "Footprint" "ProjectLocal:H_M2_GH60_MountingHole" (id 2) (at 48.26 179.07 0)
       (effects (font (size 1.27 1.27)) hide)
     )
@@
     )
     (path "/00000000-0000-0000-0000-0000602eeb15"
-      (reference "H5") (unit 1) (value "~") (footprint "ProjectLocal:H_M2_Spacer_Hole")
+      (reference "H5") (unit 1) (value "~") (footprint "ProjectLocal:H_M2_GH60_MountingHole")
     )
     (path "/00000000-0000-0000-0000-000061bfb907"
