File: pcb/keyboard-ch32x-36-lhs.kicad_sch (KiCad schematic)
At the start: 57 parts, among them J1 PJ-320A, J1 USB Type-C Receptacle 12-pin, J4 Conn_01x02, J5 Conn_01x03, SW1 SW_SPST, SW2 SW_SPST, U1 CH32X033F8P6

Commit message: pcb: save keyboard-ch32x-36-lhs with kicad9
Parts:
- renumbered J1 to J2, R1 to R5, R2 to R6
